File: pcb/sketchy.kicad_pcb (KiCad board)
At the start: 2 copper layers, 263.5 x 113.7 mm, 94 parts, among them J1 OLED, J2 OLED, SW1 SW_Push, U1 Elite-C

Commit message: Update build guide
Parts:
- moved U1 3.00 mm to (148.4, 46.7)
- moved SW1 1.59 mm to (165.1, 33.8)
- moved D108 1.59 mm to (159.5, 53.2)
Routing:
- net Col1: track 193.2 -> 202.4 mm
- net Col0: track 245.2 -> 253.7 mm, vias 6 -> 7
- net Net-(SW1-Pad1): track 18.1 -> 10.7 mm
- net Row4: track 302.6 -> 309.6 mm
- net Col7: track 86.1 -> 90.3 mm
- net RB1: track 207.6 -> 211.7 mm
- net RA1: track 196.4 -> 200.5 mm
- net Row0: track 208.5 -> 204.4 mm
- net Col2: track 136.1 -> 139.4 mm
- net Row1: track 204.7 -> 207.4 mm
- net RA2: track 213.7 -> 211.1 mm
- net SDA: track 446.5 -> 449.2 mm
- net Net-(D108-Pad1): track 17.4 -> 19.9 mm
- net Col6: track 71.2 -> 68.8 mm
- net Row3: track 258.7 -> 260.6 mm
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Other:
- outline, holes or cut-outs redrawn
- board text added: "Rev 2"
